File: I2CConnector.kicad_sch (KiCad schematic)
At the start: 10 parts, among them J5 I2C

Commit message: Initial commit.
Parts:
- removed R41: 0Ω, Resistor_SMD:R_0805_2012Metric, symbol Device:R
Connections:
- net +5V: now also D3.2 (K)
- net VBus: no longer D3.2 (K)
